File: STM32F302.kicad_sch (KiCad schematic)
At the start: 15 parts, among them SW1 SPST_SW, U2 STM32F302CBTx, Y1 12MHz

Commit message: 5/28 kicad sch
Connections:
- net CAN_RX is gone; now on net CYCLE_LED: U2.45 (PB8)
- net CYCLE_LED: no longer U2.42 (PB6)
- net TIM2_CH1: now reaches U2.10 (PA0)
- net TIM2_CH2: now reaches U2.11 (PA1)
- net MD0_DIR: now reaches U2.13 (PA3)
- net MD1_DIR: now reaches U2.14 (PA4)
- net TIM3_CH1: now reaches U2.40 (PB4)
- net TIM3_CH2: now reaches U2.41 (PB5)
- net TIM4_CH2: now reaches U2.43 (PB7)
- net CAN_TX: no longer names the net of U2.46 (PB9)
- new net TIM4_CH1: U2.42 (PB6)
- no-connect marks 20 -> 14
